Commit message: Implement and check tocabi force feedback

File: dyros_avatar_haptic_description/urdf/dyros_avatar_haptic_left.urdf (robot description, URDF)
Before this commit: robot dyros_avatar_haptic, 7 links, 6 joints
Links:
- added link base_link
Joints:
- added joint base_footprint_joint: type fixed, parent base_link, child L0v2_1, origin xyz=0 0.5 0 rpy=0 0 0

File: dyros_avatar_haptic_description/urdf/dyros_avatar_haptic_right.urdf (robot description, URDF)
Before this commit: robot dyros_avatar_haptic, 7 links, 6 joints
Links:
- added link base_link
Joints:
- added joint base_footprint_joint: type fixed, parent base_link, child R0v2_1, origin xyz=0 -0.5 1.0 rpy=0 0 0

Commit message: Check joint direction with the real robot

File: dyros_avatar_haptic_description/urdf/dyros_avatar_haptic_left.urdf (robot description, URDF)
Before this commit: robot dyros_avatar_haptic, 8 links, 7 joints
Joints:
- joint Rev2: axis 0.0 0.0 1.0 -> 0.0 0.0 -1.0
- joint Rev3: axis 0.0 0.0 1.0 -> 0.0 0.0 -1.0

File: dyros_avatar_haptic_description/urdf/dyros_avatar_haptic_right.urdf (robot description, URDF)
Before this commit: robot dyros_avatar_haptic, 8 links, 7 joints
Joints:
- joint Rev2: axis 0.0 0.0 1.0 -> 0.0 0.0 -1.0
- joint Rev3: axis 0.0 0.0 1.0 -> 0.0 0.0 -1.0
