Commit message: Update gymbol links

File: dyros_avatar_haptic_description/urdf/dyros_avatar_haptic_both.urdf (robot description, URDF)
Before this commit: robot dyros_avatar_haptic, 15 links, 14 joints
Links:
- removed link L0v2_1
- removed link L1v2_1
- removed link L4v2_1
- removed link L5v2_1
- removed link L6v2_1
- removed link R4v2_1
- removed link R5v2_1
- removed link R6v3_1
- added link L0v1_1, mass 83.96706134148887; collision mesh filename=package://dyros_avatar_haptic_description/meshes/L0v1_1_red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 scale=0.001 0.001 0.001; visual mesh filename=package://dyros_avatar_haptic_description/meshes/L0v1_1_red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 scale=0.001 0.001 0.001
- added link L1v4_1, mass 9.311307466586474; collision mesh filename=package://dyros_avatar_haptic_description/meshes/L1v4_1_red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 scale=0.001 0.001 0.001; visual mesh filename=package://dyros_avatar_haptic_description/meshes/L1v4_1_red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 scale=0.001 0.001 0.001
- added link L4v5_1, mass 2.6616567255115777; collision mesh filename=package://dyros_avatar_haptic_description/meshes/L4v5_1_red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 scale=0.001 0.001 0.001; visual mesh filename=package://dyros_avatar_haptic_description/meshes/L4v5_1_red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 scale=0.001 0.001 0.001
- added link L5v6_1, mass 1.6499764908897157; collision mesh filename=package://dyros_avatar_haptic_description/meshes/L5v6_1_red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 scale=0.001 0.001 0.001; visual mesh filename=package://dyros_avatar_haptic_description/meshes/L5v6_1_red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 scale=0.001 0.001 0.001
- added link L6v5_1, mass 0.29003290841142326; collision mesh filename=package://dyros_avatar_haptic_description/meshes/L6v5_1_red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 scale=0.001 0.001 0.001; visual mesh filename=package://dyros_avatar_haptic_description/meshes/L6v5_1_red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 scale=0.001 0.001 0.001
- added link R4v1_1, mass 2.6616567255115777; collision mesh filename=package://dyros_avatar_haptic_description/meshes/R4v1_1_red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 scale=0.001 0.001 0.001; visual mesh filename=package://dyros_avatar_haptic_description/meshes/R4v1_1_red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 scale=0.001 0.001 0.001
- added link R5v3_1, mass 1.6499764908897157; collision mesh filename=package://dyros_avatar_haptic_description/meshes/R5v3_1_red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 scale=0.001 0.001 0.001; visual mesh filename=package://dyros_avatar_haptic_description/meshes/R5v3_1_red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 scale=0.001 0.001 0.001
- added link R6v1_1, mass 0.29003290841142326; collision mesh filename=package://dyros_avatar_haptic_description/meshes/R6v1_1_red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 scale=0.001 0.001 0.001; visual mesh filename=package://dyros_avatar_haptic_description/meshes/R6v1_1_red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 scale=0.001 0.001 0.001
- link L2v2_1: mass 3.81569646652048 -> 3.7894327940262715
- link L3v2_1: mass 2.2253234887304045 -> 2.2188807496265475
- link R0v2_1: mass 96.30275269300822 -> 54.47494543793283
- link R1v2_1: mass 25.051059193207056 -> 9.600608608246226
- link R2v2_1: mass 3.7157012939377037 -> 3.6400232117451474
- link R3v2_1: mass 2.303655764107939 -> 2.275600802694944
Joints:
- joint L_Rev1: axis -1.9785965043687577e-13 4.98557253978501e-16 0.999999999999999 -> 0.0 0.0 1.0; child L1v2_1 -> L1v4_1; origin xyz=0.15434484425638284 0.04789605532138844 1.1221999999997916 rpy=0 0 0 -> xyz=1.696420781627239e-15 -6.128431095930863e-16 0.4776999999999999 rpy=0 0 0; parent L0v2_1 -> L0v1_1
- joint L_Rev2: axis -1.9809494050748165e-13 4.918921006832097e-16 0.9999999999999986 -> 0.0 0.0 1.0; origin xyz=0.25846973727083145 -0.06422191927308538 0.282100000000048 rpy=0 0 0 -> xyz=0.2585000969116214 -0.06409960917729793 0.276299999999999 rpy=0 0 0; parent L1v2_1 -> L1v4_1
- joint L_Rev3: axis 1.9816330287697064e-13 -4.919243450884573e-16 -0.999999999999999 -> 0.0 0.0 1.0; origin xyz=0.4980211697037946 0.044765103896356406 0.054300000000098825 rpy=0 0 0 -> xyz=0.49799993196454406 0.04500075291936673 0.05450000000000044 rpy=0 0 0
- joint L_Rev4: axis -1.264349999867203e-13 -1.5138091700230881e-13 -0.9999999999999986 -> 0.0 0.0 1.0; child L4v2_1 -> L4v5_1; origin xyz=0.409912459817659 -0.18569336360310523 -0.022800000000037235 rpy=0 0 0 -> xyz=0.4100002804544567 -0.18549938012637232 -0.010299999999958898 rpy=0 0 0
- joint L_Rev5: axis -0.00047166887155364285 -0.9999998887642285 -7.445754955941802e-14 -> 1.5118863886020234e-06 -0.9999999999988557 2.949330639563436e-16; child L5v2_1 -> L5v6_1; origin xyz=9.442810814563884e-05 0.20019997773060216 -0.47649999999996173 rpy=0 0 0 -> xyz=-1.3270582810420706e-07 0.08777499999989932 -0.1560749999999993 rpy=0 0 0; parent L4v2_1 -> L4v5_1
- joint L_Rev6: axis 0.9999998887642307 -0.0004716688715537389 1.5182680658618058e-13 -> 0.9999999999988606 1.5118863825447053e-06 -1.3039890257532913e-14; child L6v2_1 -> L6v5_1; origin xyz=0.3019055382987106 -0.20034242172980543 3.097522238704187e-14 rpy=0 0 0 -> xyz=-0.03719986816345422 -0.08720005624207372 1.1546319456101628e-14 rpy=0 0 0; parent L5v2_1 -> L5v6_1
- joint R_Rev1: axis 2.6367796834847473e-16 -8.320398604795848e-17 1.0000000000000007 -> 9.714451465470158e-17 -8.320398604794834e-17 1.000000000000001; origin xyz=0.06090000000000058 -0.004100000000000117 0.12220000000000049 rpy=0 0 0 -> xyz=1.2612133559741782e-15 1.8041124150158794e-16 0.47869999999999935 rpy=0 0 0
- joint R_Rev2: axis 1.1489890949413866e-15 -4.0963920219047034e-16 -1.0 -> 0.0 0.0 1.0; origin xyz=0.2585480454957062 0.06403943059620697 0.30130000000000046 rpy=0 0 0 -> xyz=0.258548045495706 0.06403943059620662 0.28680000000000094 rpy=0 0 0
- joint R_Rev3: axis -1.015837663818999e-16 -3.522754464334303e-16 -1.000000000000001 -> 0.0 0.0 1.0; origin xyz=0.49798944399048123 -0.0451166673641936 0.054500000000000104 rpy=0 0 0 -> xyz=0.49798944399048045 -0.04511666736419407 0.05449999999999955 rpy=0 0 0
- joint R_Rev4: axis 2.1372581707861384e-16 -3.967117874549952e-16 -1.000000000000002 -> 0.0 0.0 1.0; child R4v2_1 -> R4v1_1; origin xyz=0.4102030194850652 0.18505062227762256 -0.010299999999999365 rpy=0 0 0 -> xyz=0.4102030194850642 0.18505062227762417 -0.010299999999998977 rpy=0 0 0
- joint R_Rev5: axis 0.001095771599960823 0.9999993996421215 2.3141483428879694e-16 -> 0.0010957715999700898 0.9999993996421189 7.640945265029723e-16; child R5v2_1 -> R5v3_1; origin xyz=-0.0002264959897115837 -0.20669987590602634 -0.4815000000000005 rpy=0 0 0 -> xyz=-9.618135218758539e-05 -0.0877749473035866 -0.15607500000000007 rpy=0 0 0; parent R4v2_1 -> R4v1_1
- joint R_Rev6: axis 0.9999993996421225 -0.001095771599961881 3.594176539271707e-16 -> 0.9999993996421241 -0.0010957715999707956 1.2327063634757942e-14; child R6v3_1 -> R6v1_1; origin xyz=0.30822466742208654 0.2048623791537749 -1.8615317620707117e-14 rpy=0 0 0 -> xyz=-0.03790442590288334 0.08724158696959348 -4.773959005888173e-15 rpy=0 0 0; parent R5v2_1 -> R5v3_1
- joint base_footprint_joint_left: child L0v2_1 -> L0v1_1
- joint base_footprint_joint_right: origin xyz=0 -0.5 1.0 rpy=0 0 0 -> xyz=0 -0.5 0.0 rpy=0 0 0

File: dyros_avatar_haptic_description/urdf/dyros_avatar_haptic_left.urdf (robot description, URDF)
Before this commit: robot dyros_avatar_haptic, 8 links, 7 joints
Links:
- removed link L0v2_1
- removed link L1v2_1
- removed link L4v2_1
- removed link L5v2_1
- added link L0v1_1, mass 83.96706134148887; collision mesh filename=package://dyros_avatar_haptic_description/meshes/L0v1_1.stl scale=0.001 0.001 0.001; visual mesh filename=package://dyros_avatar_haptic_description/meshes/L0v1_1.stl scale=0.001 0.001 0.001
- added link L1v4_1, mass 9.311307466586474; collision mesh filename=package://dyros_avatar_haptic_description/meshes/L1v4_1.stl scale=0.001 0.001 0.001; visual mesh filename=package://dyros_avatar_haptic_description/meshes/L1v4_1.stl scale=0.001 0.001 0.001
- added link L4v5_1, mass 2.6616567255115777; collision mesh filename=package://dyros_avatar_haptic_description/meshes/L4v5_1.stl scale=0.001 0.001 0.001; visual mesh filename=package://dyros_avatar_haptic_description/meshes/L4v5_1.stl scale=0.001 0.001 0.001
- added link L5v6_1, mass 1.6499764908897157; collision mesh filename=package://dyros_avatar_haptic_description/meshes/L5v6_1.stl scale=0.001 0.001 0.001; visual mesh filename=package://dyros_avatar_haptic_description/meshes/L5v6_1.stl scale=0.001 0.001 0.001
- link EE: mass 0.5876479968624119 -> 0.29003290841142326; geometry collision mesh filename=package://dyros_avatar_haptic_description/meshes/L6v5_1.stl scale=0.001 0.001 0.001; visual mesh filename=package://dyros_avatar_haptic_description/meshes/L6v5_1.stl scale=0.001 0.001 0.001
- link L2v2_1: mass 3.81569646652048 -> 3.7894327940262715
- link L3v2_1: mass 2.2253234887304045 -> 2.2188807496265475
Joints:
- joint Rev1: axis -1.9785965043687577e-13 4.98557253978501e-16 0.999999999999999 -> 0.0 0.0 1.0; child L1v2_1 -> L1v4_1; origin xyz=0.15434484425638284 0.04789605532138844 1.1221999999997916 rpy=0 0 0 -> xyz=1.696420781627239e-15 -6.128431095930863e-16 0.4776999999999999 rpy=0 0 0; parent L0v2_1 -> L0v1_1
- joint Rev2: axis -1.9809494050748165e-13 4.918921006832097e-16 0.9999999999999986 -> 0.0 0.0 1.0; origin xyz=0.25846973727083145 -0.06422191927308538 0.282100000000048 rpy=0 0 0 -> xyz=0.2585000969116214 -0.06409960917729793 0.276299999999999 rpy=0 0 0; parent L1v2_1 -> L1v4_1
- joint Rev3: axis 1.9816330287697064e-13 -4.919243450884573e-16 -0.999999999999999 -> 0.0 0.0 1.0; origin xyz=0.4980211697037946 0.044765103896356406 0.054300000000098825 rpy=0 0 0 -> xyz=0.49799993196454406 0.04500075291936673 0.05450000000000044 rpy=0 0 0
- joint Rev4: axis -1.264349999867203e-13 -1.5138091700230881e-13 -0.9999999999999986 -> 0.0 0.0 1.0; child L4v2_1 -> L4v5_1; origin xyz=0.409912459817659 -0.18569336360310523 -0.022800000000037235 rpy=0 0 0 -> xyz=0.4100002804544567 -0.18549938012637232 -0.010299999999958898 rpy=0 0 0
- joint Rev5: axis -0.00047166887155364285 -0.9999998887642285 -7.445754955941802e-14 -> 1.5118863886020234e-06 -0.9999999999988557 2.949330639563436e-16; child L5v2_1 -> L5v6_1; origin xyz=9.442810814563884e-05 0.20019997773060216 -0.47649999999996173 rpy=0 0 0 -> xyz=-1.3270582810420706e-07 0.08777499999989932 -0.1560749999999993 rpy=0 0 0; parent L4v2_1 -> L4v5_1
- joint Rev6: axis 0.9999998887642307 -0.0004716688715537389 1.5182680658618058e-13 -> 0.9999999999988606 1.5118863825447053e-06 -1.3039890257532913e-14; origin xyz=0.3019055382987106 -0.20034242172980543 3.097522238704187e-14 rpy=0 0 0 -> xyz=-0.03719986816345422 -0.08720005624207372 1.1546319456101628e-14 rpy=0 0 0; parent L5v2_1 -> L5v6_1
- joint base_footprint_joint: child L0v2_1 -> L0v1_1

File: dyros_avatar_haptic_description/urdf/dyros_avatar_haptic_right.urdf (robot description, URDF)
Before this commit: robot dyros_avatar_haptic, 8 links, 7 joints
Links:
- removed link R4v2_1
- removed link R5v2_1
- added link R4v1_1, mass 2.6616567255115777; collision mesh filename=package://dyros_avatar_haptic_description/meshes/R4v1_1.stl scale=0.001 0.001 0.001; visual mesh filename=package://dyros_avatar_haptic_description/meshes/R4v1_1.stl scale=0.001 0.001 0.001
- added link R5v3_1, mass 1.6499764908897157; collision mesh filename=package://dyros_avatar_haptic_description/meshes/R5v3_1.stl scale=0.001 0.001 0.001; visual mesh filename=package://dyros_avatar_haptic_description/meshes/R5v3_1.stl scale=0.001 0.001 0.001
- link EE: mass 1.824291703230706 -> 0.29003290841142326; geometry collision mesh filename=package://dyros_avatar_haptic_description/meshes/R6v1_1.stl scale=0.001 0.001 0.001; visual mesh filename=package://dyros_avatar_haptic_description/meshes/R6v1_1.stl scale=0.001 0.001 0.001
- link R0v2_1: mass 96.30275269300822 -> 54.47494543793283
- link R1v2_1: mass 25.051059193207056 -> 9.600608608246226; geometry collision mesh filename=package://dyros_avatar_haptic_description/meshes/R1v2_1.stl scale=0.001 0.001 0.001; visual mesh filename=package://dyros_avatar_haptic_description/meshes/R1v2_1.stl scale=0.001 0.001 0.001
- link R2v2_1: mass 3.7157012939377037 -> 3.6400232117451474; geometry collision mesh filename=package://dyros_avatar_haptic_description/meshes/R2v2_1.stl scale=0.001 0.001 0.001; visual mesh filename=package://dyros_avatar_haptic_description/meshes/R2v2_1.stl scale=0.001 0.001 0.001
- link R3v2_1: mass 2.303655764107939 -> 2.275600802694944; geometry collision mesh filename=package://dyros_avatar_haptic_description/meshes/R3v2_1.stl scale=0.001 0.001 0.001; visual mesh filename=package://dyros_avatar_haptic_description/meshes/R3v2_1.stl scale=0.001 0.001 0.001
Joints:
- joint Rev1: axis 2.6367796834847473e-16 -8.320398604795848e-17 1.0000000000000007 -> 9.714451465470158e-17 -8.320398604794834e-17 1.000000000000001; origin xyz=0.06090000000000058 -0.004100000000000117 0.12220000000000049 rpy=0 0 0 -> xyz=1.2612133559741782e-15 1.8041124150158794e-16 0.47869999999999935 rpy=0 0 0
- joint Rev2: axis 1.1489890949413866e-15 -4.0963920219047034e-16 -1.0 -> 0.0 0.0 1.0; origin xyz=0.2585480454957062 0.06403943059620697 0.30130000000000046 rpy=0 0 0 -> xyz=0.258548045495706 0.06403943059620662 0.28680000000000094 rpy=0 0 0
- joint Rev3: axis -1.015837663818999e-16 -3.522754464334303e-16 -1.000000000000001 -> 0.0 0.0 1.0; origin xyz=0.49798944399048123 -0.0451166673641936 0.054500000000000104 rpy=0 0 0 -> xyz=0.49798944399048045 -0.04511666736419407 0.05449999999999955 rpy=0 0 0
- joint Rev4: axis 2.1372581707861384e-16 -3.967117874549952e-16 -1.000000000000002 -> 0.0 0.0 1.0; child R4v2_1 -> R4v1_1; origin xyz=0.4102030194850652 0.18505062227762256 -0.010299999999999365 rpy=0 0 0 -> xyz=0.4102030194850642 0.18505062227762417 -0.010299999999998977 rpy=0 0 0
- joint Rev5: axis 0.001095771599960823 0.9999993996421215 2.3141483428879694e-16 -> 0.0010957715999700898 0.9999993996421189 7.640945265029723e-16; child R5v2_1 -> R5v3_1; origin xyz=-0.0002264959897115837 -0.20669987590602634 -0.4815000000000005 rpy=0 0 0 -> xyz=-9.618135218758539e-05 -0.0877749473035866 -0.15607500000000007 rpy=0 0 0; parent R4v2_1 -> R4v1_1
- joint Rev6: axis 0.9999993996421225 -0.001095771599961881 3.594176539271707e-16 -> 0.9999993996421241 -0.0010957715999707956 1.2327063634757942e-14; origin xyz=0.30822466742208654 0.2048623791537749 -1.8615317620707117e-14 rpy=0 0 0 -> xyz=-0.03790442590288334 0.08724158696959348 -4.773959005888173e-15 rpy=0 0 0; parent R5v2_1 -> R5v3_1
- joint base_footprint_joint: origin xyz=0 -0.5 1.0 rpy=0 0 0 -> xyz=0 -0.5 0.0 rpy=0 0 0
