Commit message: Link 1,2,3 reduced

File: dyros_avatar_haptic_description/urdf/dyros_avatar_haptic_both.urdf (robot description, URDF)
Before this commit: robot dyros_avatar_haptic, 15 links, 14 joints
Links:
- link L2v2_1: mass 3.7894327940262715 -> 3.6056700794408694; geometry collision mesh filename=package://dyros_avatar_haptic_description/meshes/L2_Newv4_1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 scale=0.001 0.001 0.001; visual mesh filename=package://dyros_avatar_haptic_description/meshes/L2_Newv4_1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 scale=0.001 0.001 0.001
- link L3v2_1: mass 2.2188807496265475 -> 2.262098039986338; geometry collision mesh filename=package://dyros_avatar_haptic_description/meshes/L3_Newv3_1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 scale=0.001 0.001 0.001; visual mesh filename=package://dyros_avatar_haptic_description/meshes/L3_Newv3_1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 scale=0.001 0.001 0.001
- link L6v5_1: geometry collision mesh filename=package://dyros_avatar_haptic_description/meshes/L6v5_1.stl scale=0.001 0.001 0.001; visual mesh filename=package://dyros_avatar_haptic_description/meshes/L6v5_1.stl scale=0.001 0.001 0.001
- link R2v2_1: mass 3.6400232117451474 -> 3.481861325153536; geometry collision mesh filename=package://dyros_avatar_haptic_description/meshes/R2_Newv6_1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 scale=0.001 0.001 0.001; visual mesh filename=package://dyros_avatar_haptic_description/meshes/R2_Newv6_1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 scale=0.001 0.001 0.001
- link R3v2_1: mass 2.275600802694944 -> 2.298579454210347; geometry collision mesh filename=package://dyros_avatar_haptic_description/meshes/R3_Newv2_1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 scale=0.001 0.001 0.001; visual mesh filename=package://dyros_avatar_haptic_description/meshes/R3_Newv2_1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 scale=0.001 0.001 0.001
- link R6v1_1: geometry collision mesh filename=package://dyros_avatar_haptic_description/meshes/R6v1_1.stl scale=0.001 0.001 0.001; visual mesh filename=package://dyros_avatar_haptic_description/meshes/R6v1_1.stl scale=0.001 0.001 0.001
Joints:
- joint L_Rev1: origin xyz=1.696420781627239e-15 -6.128431095930863e-16 0.4776999999999999 rpy=0 0 0 -> xyz=-3.0000000002416984e-06 1.509903313490213e-16 0.478700000000001 rpy=0 0 0
- joint L_Rev2: axis 0.0 0.0 1.0 -> 0.0 0.0 -1.0; origin xyz=0.2585000969116214 -0.06409960917729793 0.276299999999999 rpy=0 0 0 -> xyz=0.2584697372708894 -0.06422191927307576 0.27629999999999943 rpy=0 0 0
- joint L_Rev3: axis 0.0 0.0 1.0 -> 0.0 0.0 -1.0; origin xyz=0.49799993196454406 0.04500075291936673 0.05450000000000044 rpy=0 0 0 -> xyz=0.3471161864898394 0.0448362810874314 0.054500000000000104 rpy=0 0 0
- joint L_Rev4: origin xyz=0.4100002804544567 -0.18549938012637232 -0.010299999999958898 rpy=0 0 0 -> xyz=0.2495124776598847 -0.18561770791609658 -0.010300000000000531 rpy=0 0 0
- joint L_Rev5: axis 1.5118863886020234e-06 -0.9999999999988557 2.949330639563436e-16 -> 0.0 1.0 0.0; origin xyz=-1.3270582810420706e-07 0.08777499999989932 -0.1560749999999993 rpy=0 0 0 -> xyz=4.140073519665055e-05 0.08777499023628024 -0.15607499999999963 rpy=0 0 0
- joint L_Rev6: axis 0.9999999999988606 1.5118863825447053e-06 -1.3039890257532913e-14 -> 1.0 0.0 0.0; origin xyz=-0.03719986816345422 -0.08720005624207372 1.1546319456101628e-14 rpy=0 0 0 -> xyz=-0.037241125387620144 -0.0871824442182206 1.7208456881689926e-14 rpy=0 0 0
- joint R_Rev1: axis 9.714451465470158e-17 -8.320398604794834e-17 1.000000000000001 -> 1.1102230246251642e-16 -3.052485909729872e-16 1.0000000000000018; origin xyz=1.2612133559741782e-15 1.8041124150158794e-16 0.47869999999999935 rpy=0 0 0 -> xyz=-3.819167204710538e-16 1.521005543736465e-16 0.4787000000000002 rpy=0 0 0
- joint R_Rev2: axis 0.0 0.0 1.0 -> 0.0 0.0 -1.0; origin xyz=0.258548045495706 0.06403943059620662 0.28680000000000094 rpy=0 0 0 -> xyz=0.2585480454957073 0.06403943059620654 0.2868000000000009 rpy=0 0 0
- joint R_Rev3: axis 0.0 0.0 1.0 -> 0.0 0.0 -1.0; origin xyz=0.49798944399048045 -0.04511666736419407 0.05449999999999955 rpy=0 0 0 -> xyz=0.3469894481342562 -0.045081291945593294 0.05449999999999977 rpy=0 0 0
- joint R_Rev4: origin xyz=0.4102030194850642 0.18505062227762417 -0.010299999999998977 rpy=0 0 0 -> xyz=0.24980311578247028 0.18522638404226016 -0.010299999999999532 rpy=0 0 0
- joint R_Rev5: axis 0.0010957715999700898 0.9999993996421189 7.640945265029723e-16 -> 0.0010957715999700898 -0.9999993996421189 7.640945265029723e-16; origin xyz=-9.618135218758539e-05 -0.0877749473035866 -0.15607500000000007 rpy=0 0 0 -> xyz=-9.618135218369961e-05 -0.08777494730358672 -0.15607500000000019 rpy=0 0 0
- joint R_Rev6: origin xyz=-0.03790442590288334 0.08724158696959348 -4.773959005888173e-15 rpy=0 0 0 -> xyz=-0.03790442590288501 0.08724158696959274 -4.440892098500626e-15 rpy=0 0 0

File: dyros_avatar_haptic_description/urdf/dyros_avatar_haptic_left.urdf (robot description, URDF)
Before this commit: robot dyros_avatar_haptic, 8 links, 7 joints
Links:
- link L2v2_1: mass 3.7894327940262715 -> 3.6056700794408694; geometry collision mesh filename=package://dyros_avatar_haptic_description/meshes/L2_Newv4_1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 scale=0.001 0.001 0.001; visual mesh filename=package://dyros_avatar_haptic_description/meshes/L2_Newv4_1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 scale=0.001 0.001 0.001
- link L3v2_1: mass 2.2188807496265475 -> 2.262098039986338; geometry collision mesh filename=package://dyros_avatar_haptic_description/meshes/L3_Newv3_1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 scale=0.001 0.001 0.001; visual mesh filename=package://dyros_avatar_haptic_description/meshes/L3_Newv3_1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 scale=0.001 0.001 0.001
Joints:
- removed joint Rev1
- removed joint Rev2
- removed joint Rev3
- removed joint Rev4
- removed joint Rev5
- removed joint Rev6
- added joint L_Rev1: type prismatic, parent L0v1_1, child L1v4_1, origin xyz=-3.0000000002416984e-06 1.509903313490213e-16 0.478700000000001 rpy=0 0 0, axis 0.0 0.0 1.0, limit lower=-3.14159 upper=3.14159 effort=100 velocity=100
- added joint L_Rev2: type revolute, parent L1v4_1, child L2v2_1, origin xyz=0.2584697372708894 -0.06422191927307576 0.27629999999999943 rpy=0 0 0, axis 0.0 0.0 -1.0, limit lower=-3.14159 upper=3.14159 effort=100 velocity=100
- added joint L_Rev3: type revolute, parent L2v2_1, child L3v2_1, origin xyz=0.3471161864898394 0.0448362810874314 0.054500000000000104 rpy=0 0 0, axis 0.0 0.0 -1.0, limit lower=-3.14159 upper=3.14159 effort=100 velocity=100
- added joint L_Rev4: type revolute, parent L3v2_1, child L4v5_1, origin xyz=0.2495124776598847 -0.18561770791609658 -0.010300000000000531 rpy=0 0 0, axis 0.0 0.0 1.0, limit lower=-3.14159 upper=3.14159 effort=100 velocity=100
- added joint L_Rev5: type revolute, parent L4v5_1, child L5v6_1, origin xyz=4.140073519665055e-05 0.08777499023628024 -0.15607499999999963 rpy=0 0 0, axis 0.0 1.0 0.0, limit lower=-3.14159 upper=3.14159 effort=100 velocity=100
- added joint L_Rev6: type revolute, parent L5v6_1, child EE, origin xyz=-0.037241125387620144 -0.0871824442182206 1.7208456881689926e-14 rpy=0 0 0, axis 1.0 0.0 0.0, limit lower=-3.14159 upper=3.14159 effort=100 velocity=100

File: dyros_avatar_haptic_description/urdf/dyros_avatar_haptic_right.urdf (robot description, URDF)
Before this commit: robot dyros_avatar_haptic, 8 links, 7 joints
Links:
- link R2v2_1: mass 3.6400232117451474 -> 3.481861325153536; geometry collision mesh filename=package://dyros_avatar_haptic_description/meshes/R2_Newv6_1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 scale=0.001 0.001 0.001; visual mesh filename=package://dyros_avatar_haptic_description/meshes/R2_Newv6_1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 scale=0.001 0.001 0.001
- link R3v2_1: mass 2.275600802694944 -> 2.298579454210347; geometry collision mesh filename=package://dyros_avatar_haptic_description/meshes/R3_Newv2_1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 scale=0.001 0.001 0.001; visual mesh filename=package://dyros_avatar_haptic_description/meshes/R3_Newv2_1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 scale=0.001 0.001 0.001
Joints:
- removed joint Rev1
- removed joint Rev2
- removed joint Rev3
- removed joint Rev4
- removed joint Rev5
- removed joint Rev6
- added joint R_Rev1: type prismatic, parent R0v2_1, child R1v2_1, origin xyz=-3.819167204710538e-16 1.521005543736465e-16 0.4787000000000002 rpy=0 0 0, axis 1.1102230246251642e-16 -3.052485909729872e-16 1.0000000000000018, limit lower=-3.14159 upper=3.14159 effort=100 velocity=100
- added joint R_Rev2: type revolute, parent R1v2_1, child R2v2_1, origin xyz=0.2585480454957073 0.06403943059620654 0.2868000000000009 rpy=0 0 0, axis 0.0 0.0 -1.0, limit lower=-3.14159 upper=3.14159 effort=100 velocity=100
- added joint R_Rev3: type revolute, parent R2v2_1, child R3v2_1, origin xyz=0.3469894481342562 -0.045081291945593294 0.05449999999999977 rpy=0 0 0, axis 0.0 0.0 -1.0, limit lower=-3.14159 upper=3.14159 effort=100 velocity=100
- added joint R_Rev4: type revolute, parent R3v2_1, child R4v1_1, origin xyz=0.24980311578247028 0.18522638404226016 -0.010299999999999532 rpy=0 0 0, axis 0.0 0.0 1.0, limit lower=-3.14159 upper=3.14159 effort=100 velocity=100
- added joint R_Rev5: type revolute, parent R4v1_1, child R5v3_1, origin xyz=-9.618135218369961e-05 -0.08777494730358672 -0.15607500000000019 rpy=0 0 0, axis 0.0010957715999700898 -0.9999993996421189 7.640945265029723e-16, limit lower=-3.14159 upper=3.14159 effort=100 velocity=100
- added joint R_Rev6: type revolute, parent R5v3_1, child EE, origin xyz=-0.03790442590288501 0.08724158696959274 -4.440892098500626e-15 rpy=0 0 0, axis 0.9999993996421241 -0.0010957715999707956 1.2327063634757942e-14, limit lower=-3.14159 upper=3.14159 effort=100 velocity=100
